File: frdm05-devboard-hardware/frdm05-devboard.kicad_pcb (KiCad board)
At the start: 2 copper layers, 99.1 x 84.8 mm, 63 parts, among them CON1 MIKROBUS_HOST_CONN, J1 SD_Card_Fix, J2 KEYBOARD, J3 Conn_01x06, J4 LIGHT SENSOR, J5 1602 LCD VIA I2C, Q1 BCV62, Q2 BC817, SW1 PTS810, SW2 PTS810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

Commit message: Initial commit of Rev.2 hardware
Parts:
- added C10: 100n, Capacitor_SMD:C_0805_2012Metric_Pad1.18x1.45mm_HandSolder, B.Cu at (152.9, 109.2)
- added C11: 100n, Capacitor_SMD:C_0805_2012Metric_Pad1.18x1.45mm_HandSolder, B.Cu at (152.9, 100.3)
- added C7: 1u, Capacitor_SMD:C_0805_2012Metric_Pad1.18x1.45mm_HandSolder, F.Cu at (134.4, 97.0)
- added C8: 100n, Capacitor_SMD:C_0805_2012Metric_Pad1.18x1.45mm_HandSolder, B.Cu at (118.7, 77.1)
- added C9: 100n, Capacitor_SMD:C_0805_2012Metric_Pad1.18x1.45mm_HandSolder, F.Cu at (155.1, 65.8)
- added F1: Polyfuse, Fuse:Fuse_0805_2012Metric, F.Cu at (124.2, 125.0)
- added F2: Polyfuse, Fuse:Fuse_0805_2012Metric, B.Cu at (125.7, 116.3)
- added R19: 470, Resistor_SMD:R_0805_2012Metric_Pad1.20x1.40mm_HandSolder, B.Cu at (185.2, 70.9)
- moved R4 2.03 mm to (109.7, 134.1)
- moved R5 2.03 mm to (107.7, 134.1)
- moved C2 0.82 mm to (145.5, 84.5)
- moved D4 0.17 mm to (151.5, 82.5)
- moved C6 0.11 mm to (132.3, 97.0)
Connections:
- A1 pad 4: +3V3 -> Net-(A1-Pad4)
- A1 pad 5: +5V -> Net-(A1-Pad5)
- BZ1 pad 1: +5V -> Net-(BZ1-Pad1)
- Q1 pad 1: AN_KEYPAD -> Net-(Q1-Pad1)
- Q1 pad 2: Net-(Q1-Pad2) -> AN_KEYPAD
- R4 pad 1: Net-(Q1-Pad2) -> Net-(Q1-Pad1)
Routing:
- net +5V: track 201.6 -> 196.2 mm
- net Net-(A1-Pad5): track 0.00 -> 4.65 mm
- net AN_KEYPAD: track 66.7 -> 70.9 mm
- net Net-(BZ1-Pad1): track 0.00 -> 3.56 mm
- net SPI_MOSI: track 185.3 -> 182.0 mm
- net Net-(Q1-Pad1): track 0.00 -> 3.34 mm
- net Net-(Q1-Pad2): track 3.26 -> 0.00 mm
- net Net-(TP5-Pad1): track 23.9 -> 27.1 mm
- net Net-(A1-Pad4): track 0.00 -> 3.08 mm
- net I2C_SCL: track 190.4 -> 193.0 mm
- net Net-(D3-Pad2): track 7.27 -> 4.71 mm
- net +3V3: track 307.8 -> 305.6 mm, vias 12 -> 8
- net SPI_SS_SDCARD: track 36.4 -> 34.6 mm
- net SPI_MISO: track 194.0 -> 192.6 mm
- net SPI_CLK: track 198.7 -> 200.1 mm
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Other:
- board text added: "Touch with alligator clip end"
- board text removed: "Touch with aligator clip end"

Commit message: Initial commit of Rev.2.1 hardware
Parts:
- BZ1: footprint Buzzer_Beeper:Buzzer_12x9.5RM7.6 -> Buzzer_Beeper:MagneticBuzzer_ProSignal_ABT-410-RC
- C9, F1: moved to B.Cu
- moved F1 3.56 mm to (120.7, 125.1), turned to 270 degrees
- moved C9 0.64 mm to (154.4, 65.9)
Connections:
- A1 pad 2: +3V3 -> 3V3_UNPROT
- A1 pad 4: Net-(A1-Pad4) -> 3V3_UNPROT
- F1 pad 1: Net-(A1-Pad4) -> 3V3_UNPROT
Routing:
- net 3V3_UNPROT: track 0.00 -> 8.05 mm
- net +3V3: track 305.6 -> 302.4 mm, vias 8 -> 9
- net Net-(A1-Pad4): track 3.08 -> 0.00 mm
- net Net-(BZ1-Pad2): track 11.7 -> 12.8 mm
- net GND: vias 51 -> 50
Other:
- board text added: "Connect alligator clip here"
- board text removed: "Connect aligator clip here"

Commit message: Initial commit of Rev.2.2 hardware
Parts:
- U6: value 74HCT1G125GV -> 74AHCT1G125GV
